Commit message: feat(isaac): 씬 정합, 브릿지 스크립트 복구 로직, 뷰포트 HUD
USD: 보드 810mm·1500x900 콜라이더, 딸기 12개(익은 6/안 익은 6) 분면 배치, 줄기 파단력 상향,
드라이브 게인, 커스텀 파츠 6도 보정, 분면 하이라이트 오버레이.
isaac_sim_script_editor_bridge.py: 물리 스텝 콜백에서 apply_action 실패 시 재초기화·재시도,
상태 발행 분리(콜백 사망과 팔 정지 구분).
HUD(isaac_sim_hud.py + hud/): 노드 램프·영역·단계·카운터, 직전 런 잔상 무시(EPOCH).

Co-Authored-By: Claude Fable 5.1 <noreply@anthropic.com>

File: robot.urdf (robot description, URDF)
Before this commit: robot strawberry_grasp_robot, 15 links, 14 joints
Links:
- link base_link: geometry collision mesh filename=/home/oceanshape/strawberry_grasp_environment/src/doosan_ro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 scale=0.001 0.001 0.001; visual mesh filename=/home/oceanshape/strawberry_grasp_environment/src/doosan_ro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 scale=0.001 0.001 0.001
- link left_custom_part: geometry visual mesh filename=/home/oceanshape/strawberry_grasp_environment/src/strawberr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 scale=0.001 0.001 0.001
- link link_1: geometry collision mesh filename=/home/oceanshape/strawberry_grasp_environment/src/doosan_ro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 scale=0.001 0.001 0.001; collision mesh filename=/home/oceanshape/strawberry_grasp_environment/src/doosan_ro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 scale=0.001 0.001 0.001
- link link_2: geometry collision mesh filename=/home/oceanshape/strawberry_grasp_environment/src/doosan_ro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 scale=0.001 0.001 0.001; collision mesh filename=/home/oceanshape/strawberry_grasp_environment/src/doosan_ro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 scale=0.001 0.001 0.001
- link link_3: geometry collision mesh filename=/home/oceanshape/strawberry_grasp_environment/src/doosan_ro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 scale=0.001 0.001 0.001; collision mesh filename=/home/oceanshape/strawberry_grasp_environment/src/doosan_ro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 scale=0.001 0.001 0.001
- link link_4: geometry collision mesh filename=/home/oceanshape/strawberry_grasp_environment/src/doosan_ro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 scale=0.001 0.001 0.001; collision mesh filename=/home/oceanshape/strawberry_grasp_environment/src/doosan_ro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 scale=0.001 0.001 0.001
- link link_5: geometry collision mesh filename=/home/oceanshape/strawberry_grasp_environment/src/doosan_ro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 scale=0.001 0.001 0.001; collision mesh filename=/home/oceanshape/strawberry_grasp_environment/src/doosan_ro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 scale=0.001 0.001 0.001
- link link_6: geometry collision mesh filename=/home/oceanshape/strawberry_grasp_environment/src/doosan_ro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 scale=0.001 0.001 0.001; visual mesh filename=/home/oceanshape/strawberry_grasp_environment/src/doosan_ro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 scale=0.001 0.001 0.001
- link rh_p12_rn_base: geometry collision mesh filename=/home/oceanshape/strawberry_grasp_environment/src/RH-P12-RN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 scale=0.001 0.001 0.001; visual mesh filename=/home/oceanshape/strawberry_grasp_environment/src/RH-P12-RN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 scale=0.001 0.001 0.001
- link rh_p12_rn_l1: geometry collision mesh filename=/home/oceanshape/strawberry_grasp_environment/src/RH-P12-RN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 scale=0.001 0.001 0.001; visual mesh filename=/home/oceanshape/strawberry_grasp_environment/src/RH-P12-RN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 scale=0.001 0.001 0.001
- link rh_p12_rn_l2: geometry collision mesh filename=/home/oceanshape/strawberry_grasp_environment/src/RH-P12-RN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 scale=0.001 0.001 0.001; visual mesh filename=/home/oceanshape/strawberry_grasp_environment/src/RH-P12-RN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 scale=0.001 0.001 0.001
- link rh_p12_rn_r1: geometry collision mesh filename=/home/oceanshape/strawberry_grasp_environment/src/RH-P12-RN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 scale=0.001 0.001 0.001; visual mesh filename=/home/oceanshape/strawberry_grasp_environment/src/RH-P12-RN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 scale=0.001 0.001 0.001
- link rh_p12_rn_r2: geometry collision mesh filename=/home/oceanshape/strawberry_grasp_environment/src/RH-P12-RN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 scale=0.001 0.001 0.001; visual mesh filename=/home/oceanshape/strawberry_grasp_environment/src/RH-P12-RN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 scale=0.001 0.001 0.001
- link right_custom_part: geometry visual mesh filename=/home/oceanshape/strawberry_grasp_environment/src/strawberr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 scale=0.001 0.001 0.001
Joints:
- joint l2_to_left_custom_part: origin xyz=0.02090 0.00498 0.00058 rpy=-1.5707963267948966 0.10471975511965978 -1.5707963267948966 -> xyz=0.02090 0.00498 0.00058 rpy=-1.5707963267948966 0 -1.5707963267948966
- joint r2_to_right_custom_part: origin xyz=-0.02090 -0.00499 0.00058 rpy=1.5707963267948966 0.10471975511965978 1.5707963267948966 -> xyz=-0.02090 -0.00499 0.00058 rpy=1.5707963267948966 0 1.5707963267948966
- joint world_fixed: child base_link -> rh_p12_rn_base

File: src/strawberry_grasp_environment_description/urdf/robot.urdf.xacro (robot description, xacro)
@@ -4,10 +4,10 @@
   <!-- 1. Include Doosan e0509                    -->
   <!-- ========================================== -->
-  <xacro:include filename="/home/sun/strawberry_grasp_environment/src/doosan_robot2/dsr_description2/xacro/e0509.urdf.xacro" />
+  <xacro:include filename="/home/oceanshape/strawberry_grasp_environment/src/doosan_robot2/dsr_description2/xacro/e0509.urdf.xacro" />
   <!-- ========================================== -->
   <!-- 2. Include Robotis RH-P12-RN               -->
   <!-- ========================================== -->
   <!-- We modified the original file to remove the world_fixed joint -->
-  <xacro:include filename="/home/sun/strawberry_grasp_environment/src/RH-P12-RN/rh_p12_rn_description/urdf/rh_p12_rn.xacro" />
+  <xacro:include filename="/home/oceanshape/strawberry_grasp_environment/src/RH-P12-RN/rh_p12_rn_description/urdf/rh_p12_rn.xacro" />
   <!-- define pi -->
   <xacro:property name="pi" value="3.1415926535897931" />

Commit message: fix(spec): 시뮬이 실기·공식 제원보다 관대한 곳을 없앤다 — 스윙 가드 원복, 브릿지 C1~C3, 로봇 한계 D1, 가속도 D3
실기 플래너 (원복만, 규칙 §0-1: 실기 노드 수정 사유는 핵심 시퀀스 설계 불일치뿐)
- harvest_motion_params.py: MAX_HARVEST_JOINT_DELTA_DEG J1 95→75, MAX_TAUGHT_PLACE_TRANSFER J2 130→100·J3 175→120 (09-08·09-10 상향분 원본으로)

시뮬 브릿지 (본인 구현)
- C1 ARM_JOINT_LIMIT_DEG 365/160 → 공식 URDF 360/155, D1 로 J2 95·J3 135·J5 135 (실기 cuRobo 운용 값)
- C2 move_joint_cb: 즉시 발행 → 요청 vel/acc 사다리꼴 프로파일 movej_profile() (동기 이동, time 우선, 기본 60/60)
- C3 sim_speed_scale 기본 2.0 → 1.0 (실기 요청 시간 = 실행 시간)
- D3 두산 MoveIt joint_limits.yaml 참조값을 자르지 않고 초과만 기록 (DOOSAN_MOVEIT_REF / MOVEJ_OVER_DOOSAN_MOVEIT)

시뮬 로봇 모델
- robot.urdf·robot.usd: J2 ±360→±95, J3 ±155→±135, J5 ±360→±135 (실기 값; 씬 재로드 필요). 속도 180/225 는 실기와 동일 유지 (D2)

Co-Authored-By: Claude Fable 5.1 <noreply@anthropic.com>

File: robot.urdf (robot description, URDF)
Before this commit: robot strawberry_grasp_environment_robot, 15 links, 14 joints
Joints:
- joint joint_2: limit lower=-6.2832 upper=6.2832 effort=194 velocity=3.1416 -> lower=-1.6581 upper=1.6581 effort=194 velocity=3.1416
- joint joint_3: limit lower=-2.7053 upper=2.7053 effort=194 velocity=3.1416 -> lower=-2.3562 upper=2.3562 effort=194 velocity=3.1416
- joint joint_5: limit lower=-6.2832 upper=6.2832 effort=66 velocity=3.927 -> lower=-2.3562 upper=2.3562 effort=66 velocity=3.927
